File: heartPCB.kicad_pcb (KiCad board)
At the start: 2 copper layers, 69.1 x 63.7 mm, 34 parts, among them SW1 SW_SPDT, U2 4017, U4 ICM7555xP

Commit message: readme update
Parts:
- C11: value 3.3uF -> 10uF
- RC2: value 10K -> 2K
- U2: footprint Package_DIP:DIP-16_W7.62mm_Socket_LongPads -> Package_DIP:DIP-16_W7.62mm_LongPads
Changed lines of the file:
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@@
 		(property ki_fp_filters "R_*")
 		(sheetname "/")
-		(sheetfile "pcb2.kicad_sch")
+		(sheetfile "heartPCB.kicad_sch")
 		(attr through_hole)
 		(fp_line
@@
 		(property ki_fp_filters "LED* LED_SMD:* LED_THT:*")
 		(sheetname "/")
-		(sheetfile "pcb2.kicad_sch")
+		(sheetfile "heartPCB.kicad_sch")
 		(attr through_hole)
 		(fp_line
@@
 		(property ki_fp_filters "LED* LED_SMD:* LED_THT:*")
 		(sheetname "/")
-		(sheetfile "pcb2.kicad_sch")
+		(sheetfile "heartPCB.kicad_sch")
 		(attr through_hole)
 		(fp_line
@@
 			)
 		)
-		(property "Value" "10K"
+		(property "Value" "2K"
 			(at -2.39 0.8 90)
 			(layer "F.Fab")
@@
 		(property ki_fp_filters "R_*")
 		(sheetname "/")
-		(sheetfile "pcb2.kicad_sch")
+		(sheetfile "heartPCB.kicad_sch")
 		(attr through_hole)
 		(fp_line
@@
 		(property ki_fp_filters "LED* LED_SMD:* LED_THT:*")
 		(sheetname "/")
-		(sheetfile "pcb2.kicad_sch")
+		(sheetfile "heartPCB.kicad_sch")
 		(attr through_hole)
 		(fp_line
@@
 		(property ki_fp_filters "LED* LED_SMD:* LED_THT:*")
 		(sheetname "/")
-		(sheetfile "pcb2.kicad_sch")
+		(sheetfile "heartPCB.kicad_sch")
 		(attr through_hole)
 		(fp_line
@@
 		(property ki_fp_filters "C_*")
 		(sheetname "/")
-		(sheetfile "pcb2.kicad_sch")
+		(sheetfile "heartPCB.kicad_sch")
 		(attr through_hole)
 		(fp_line
@@
 		(property ki_fp_filters "R_*")
 		(sheetname "/")
-		(sheetfile "pcb2.kicad_sch")
+		(sheetfile "heartPCB.kicad_sch")
 		(attr through_hole)
 		(fp_line
@@
 		(property ki_fp_filters "R_*")
 		(sheetname "/")
-		(sheetfile "pcb2.kicad_sch")
+		(sheetfile "heartPCB.kicad_sch")
 		(attr through_hole)
 		(fp_line
@@
 		(property ki_fp_filters "LED* LED_SMD:* LED_THT:*")
 		(sheetname "/")
-		(sheetfile "pcb2.kicad_sch")
+		(sheetfile "heartPCB.kicad_sch")
 		(attr through_hole)
 		(fp_line
@@
 		(property ki_fp_filters "R_*")
 		(sheetname "/")
-		(sheetfile "pcb2.kicad_sch")
+		(sheetfile "heartPCB.kicad_sch")
 		(attr through_hole)
 		(fp_line
@@
 		(property ki_fp_filters "LED* LED_SMD:* LED_THT:*")
 		(sheetname "/")
-		(sheetfile "pcb2.kicad_sch")
+		(sheetfile "heartPCB.kicad_sch")
 		(attr through_hole)
 		(fp_line
@@
 		(property ki_fp_filters "R_*")
 		(sheetname "/")
-		(sheetfile "pcb2.kicad_sch")
+		(sheetfile "heartPCB.kicad_sch")
 		(attr through_hole)
 		(fp_line
@@
 		(property ki_fp_filters "DIP*W7.62mm*")
 		(sheetname "/")
-		(sheetfile "pcb2.kicad_sch")
+		(sheetfile "heartPCB.kicad_sch")
 		(attr through_hole)
 		(fp_line
@@
 		)
 	)
-	(footprint "Package_DIP:DIP-16_W7.62mm_Socket_LongPads"
+	(footprint "Package_DIP:DIP-16_W7.62mm_LongPads"
 		(layer "F.Cu")
 		(at 150.241 52.832)
-		(descr "16-lead though-hole mounted DIP package, row spacing 7.62mm (300 mils), Socket, LongPads")
-		(tags "THT DIP DIL PDIP 2.54mm 7.62mm 300mil Socket LongPads")
+		(descr "16-lead though-hole mounted DIP package, row spacing 7.62mm (300 mils), LongPads")
+		(tags "THT DIP DIL PDIP 2.54mm 7.62mm 300mil LongPads")
 		(property "Reference" "U2"
 			(at 3.81 -2.33 0)
@@
 		(property ki_fp_filters "DIP?16*")
 		(sheetname "/")
-		(sheetfile "pcb2.kicad_sch")
+		(sheetfile "heartPCB.kicad_sch")
 		(attr through_hole)
 		(fp_line
@@
 			(layer "F.SilkS")
 		)
-		(fp_rect
-			(start -1.44 -1.39)
-			(end 9.06 19.17)
-			(stroke
-				(width 0.12)
-				(type solid)
-			)
-			(fill no)
-			(layer "F.SilkS")
-		)
 		(fp_arc
 			(start 4.81 -1.33)
@@
 		)
 		(fp_rect
-			(start -1.52 -1.58)
-			(end 9.14 19.36)
+			(start -1.45 -1.52)
+			(end 9.07 19.3)
 			(stroke
 				(width 0.05)
@@
 			(layer "F.Fab")
 		)
-		(fp_rect
-			(start -1.27 -1.33)
-			(end 8.89 19.11)
-			(stroke
-				(width 0.1)
-				(type solid)
-			)
-			(fill no)
-			(layer "F.Fab")
-		)
 		(fp_text user "${REFERENCE}"
 			(at 3.81 8.89 90)
@@
 		)
 		(embedded_fonts no)
-		(model "${KICAD9_3DMODEL_DIR}/Package_DIP.3dshapes/DIP-16_W7.62mm_Socket.step"
+		(model "${KICAD9_3DMODEL_DIR}/Package_DIP.3dshapes/DIP-16_W7.62mm.step"
 			(offset
 				(xyz 0 0 0)
@@
 		(property ki_fp_filters "LED* LED_SMD:* LED_THT:*")
 		(sheetname "/")
-		(sheetfile "pcb2.kicad_sch")
+		(sheetfile "heartPCB.kicad_sch")
 		(attr through_hole)
 		(fp_line
@@
 		(property ki_fp_filters "LED* LED_SMD:* LED_THT:*")
 		(sheetname "/")
-		(sheetfile "pcb2.kicad_sch")
+		(sheetfile "heartPCB.kicad_sch")
 		(attr through_hole)
 		(fp_line
@@
 		(property ki_fp_filters "R_*")
 		(sheetname "/")
-		(sheetfile "pcb2.kicad_sch")
+		(sheetfile "heartPCB.kicad_sch")
 		(attr through_hole)
 		(fp_line
@@
 		(property ki_fp_filters "R_*")
 		(sheetname "/")
-		(sheetfile "pcb2.kicad_sch")
+		(sheetfile "heartPCB.kicad_sch")
 		(attr through_hole)
 		(fp_line
@@
 		(property ki_fp_filters "R_*")
 		(sheetname "/")
-		(sheetfile "pcb2.kicad_sch")
+		(sheetfile "heartPCB.kicad_sch")
 		(attr through_hole)
 		(fp_line
@@
 		(property ki_fp_filters "R_*")
 		(sheetname "/")
-		(sheetfile "pcb2.kicad_sch")
+		(sheetfile "heartPCB.kicad_sch")
 		(attr through_hole)
 		(fp_line
@@
 		(property ki_fp_filters "LED* LED_SMD:* LED_THT:*")
 		(sheetname "/")
-		(sheetfile "pcb2.kicad_sch")
+		(sheetfile "heartPCB.kicad_sch")
 		(attr through_hole)
 		(fp_line
@@
 			)
 		)
-		(property "Value" "3.3uF"
+		(property "Value" "10uF"
 			(at 1.05 4.7 0)
 			(layer "F.Fab")
@@
 		(property ki_fp_filters "CP_*")
 		(sheetname "/")
-		(sheetfile "pcb2.kicad_sch")
+		(sheetfile "heartPCB.kicad_sch")
 		(attr through_hole)
 		(fp_line
@@
 		(property ki_fp_filters "LED* LED_SMD:* LED_THT:*")
 		(sheetname "/")
-		(sheetfile "pcb2.kicad_sch")
+		(sheetfile "heartPCB.kicad_sch")
 		(attr through_hole)
 		(fp_line
@@
 		)
 		(sheetname "/")
-		(sheetfile "pcb2.kicad_sch")
+		(sheetfile "heartPCB.kicad_sch")
 		(attr through_hole)
 		(fp_rect
@@
 		(property ki_fp_filters "R_*")
 		(sheetname "/")
-		(sheetfile "pcb2.kicad_sch")
+		(sheetfile "heartPCB.kicad_sch")
 		(attr through_hole)
 		(fp_line
@@
 		(property ki_fp_filters "R_*")
 		(sheetname "/")
-		(sheetfile "pcb2.kicad_sch")
+		(sheetfile "heartPCB.kicad_sch")
 		(attr through_hole)
 		(fp_line
@@
 		(property ki_fp_filters "R_*")
 		(sheetname "/")
-		(sheetfile "pcb2.kicad_sch")
+		(sheetfile "heartPCB.kicad_sch")
 		(attr through_hole)
 		(fp_line
@@
 		(property ki_fp_filters "LED* LED_SMD:* LED_THT:*")
 		(sheetname "/")
-		(sheetfile "pcb2.kicad_sch")
+		(sheetfile "heartPCB.kicad_sch")
 		(attr through_hole)
 		(fp_line
@@
 		(property ki_fp_filters "R_*")
 		(sheetname "/")
-		(sheetfile "pcb2.kicad_sch")
+		(sheetfile "heartPCB.kicad_sch")
 		(attr through_hole)
 		(fp_line
@@
 		(property ki_fp_filters "LED* LED_SMD:* LED_THT:*")
 		(sheetname "/")
-		(sheetfile "pcb2.kicad_sch")
+		(sheetfile "heartPCB.kicad_sch")
 		(attr through_hole)
 		(fp_line
@@
 		)
 		(sheetname "/")
-		(sheetfile "pcb2.kicad_sch")
+		(sheetfile "heartPCB.kicad_sch")
 		(attr smd)
 		(fp_line
