File: heartPCB.kicad_sch (KiCad schematic)
At the start: 32 parts, among them SW1 SW_SPDT, U2 4017, U4 ICM7555xP

Commit message: schematic footprint changes
Parts:
- C11: value 3.3uF -> 2.2uF
- RC2: value 10K -> 22K
Changed lines of the file:
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@@
 			)
 		)
-		(property "Value" "10K"
+		(property "Value" "22K"
 			(at 96.52 60.9599 0)
 			(effects
@@
 			)
 		)
-		(property "Value" "3.3uF"
+		(property "Value" "2.2uF"
 			(at 110.49 71.5009 0)
 			(effects

Commit message: readme update
Parts:
- C11: value 2.2uF -> 10uF
- C12: footprint Capacitor_THT:C_Disc_D5.0mm_W2.5mm_P5.00mm -> Capacitor_THT:C_Disc_D5.0mm_W2.5mm_P2.50mm
- RC2: value 22K -> 2K
- U2: footprint Package_DIP:DIP-16_W7.62mm_Socket_LongPads -> Package_DIP:DIP-16_W7.62mm_LongPads
Changed lines of the file:
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@@
 			)
 		)
-		(property "Footprint" "Capacitor_THT:C_Disc_D5.0mm_W2.5mm_P5.00mm"
+		(property "Footprint" "Capacitor_THT:C_Disc_D5.0mm_W2.5mm_P2.50mm"
 			(at 138.1252 80.01 0)
 			(effects
@@
 			)
 		)
-		(property "Value" "22K"
+		(property "Value" "2K"
 			(at 96.52 60.9599 0)
 			(effects
@@
 			)
 		)
-		(property "Value" "2.2uF"
+		(property "Value" "10uF"
 			(at 110.49 71.5009 0)
 			(effects
@@
 			)
 		)
-		(property "Footprint" "Package_DIP:DIP-16_W7.62mm_Socket_LongPads"
+		(property "Footprint" "Package_DIP:DIP-16_W7.62mm_LongPads"
 			(at 161.29 63.5 0)
 			(effects
